File: relay_block_cryo.kicad_sch (KiCad schematic)
At the start: 16 parts, among them J1 12v, J2 HE_compressor, J4 mcu, J5 x, K1 Relay_DPDT, K2 ADW11, Q1 BC327, U1 EL817

Commit message: modified
Parts:
- removed J1: 12v, symbol Connector:Screw_Terminal_01x02
- removed J2: HE_compressor, symbol Connector:Screw_Terminal_01x02
- removed J4: mcu, symbol Connector:Screw_Terminal_01x02
- removed J5: x, symbol Connector:Screw_Terminal_01x02
- removed K1: Relay_DPDT, symbol Relay:Relay_DPDT
- removed K2: ADW11, Relay_THT:Relay_SPST_Panasonic_ADW11, symbol Relay:ADW11
- added D3: RED, symbol Device:LED_Small
- added D4: 1n4001, Diode_THT:D_DO-41_SOD81_P7.62mm_Horizontal, symbol Device:D_Small
- added H1, H2, H3, H4: MountingHole, MountingHole:MountingHole_3.2mm_M3, symbol Mechanical:MountingHole
- added J1: Phase_IN, symbol Connector:Screw_Terminal_01x01
- added J2: he_compressor, symbol Connector:Screw_Terminal_01x01
- added J3: vacuum_valve, symbol Connector:Screw_Terminal_01x01
- added J8: DB9_Female, symbol Connector_self:DB9_Female
- added K1, K3: G5V-1, Relay_THT:Relay_SPDT_Omron_G5V-1, symbol Relay:G5V-1
- added Q2: BC327, Package_TO_SOT_THT:TO-92_Inline, symbol Transistor_BJT:BC327
- added R5, R6: 22k, Resistor_SMD:R_1206_3216Metric, symbol Device:R_Small
- added R7: 5.1k, Resistor_SMD:R_1206_3216Metric, symbol Device:R_Small
- added R8: 1k, Resistor_SMD:R_1206_3216Metric, symbol Device:R_Small
- added U2: PC817, Package_DIP:DIP-4_W7.62mm, symbol Isolator:EL817
- C1, C2, R1, R2, R3, R4: footprint (none) -> Resistor_SMD:R_1206_3216Metric
- D1: footprint (none) -> Diode_THT:D_DO-41_SOD81_P7.62mm_Horizontal
- U1: value EL817 -> PC817
Connections:
- net 230VAC_F is gone; now on net 230V_F: C1.1
- net +12V: now also J8.7, Q2.1 (C), R6.1
- net 230V_F: now also J1.1 (Pin_1), K1.10, K3.10
- net GND: now also D3.1 (K), D4.2 (A), J8.3, J8.4, J8.5, J8.8, J8.9, K1.9, K3.9, U2.3
- net GND_MCU: now also J8.2, U2.2
- net at D1.1 (K), Q1.3 (E), R4.1: now also K3.2
- net 230V_FOUT1: now reaches C1.2
- net 230V_FOUT1: now also J2.1 (Pin_1), K3.5, K3.6
- net 5V_MCU renamed HEC
- net HEC: now also J8.1
- net COM_IN renamed 230V_FOUT2
- net 230V_FOUT2: now also J3.1 (Pin_1), K1.5, K1.6
- new net: D3.2 (A), R8.2
- new net: D4.1 (K), K1.2, Q2.3 (E), R8.1
- new net: R5.2, U2.1
- new net: R7.2, U2.4
- new net: Q2.2 (B), R6.2, R7.1
- new net VAS: J8.6
- new net VAV: R5.1
- no-connect marks 0 -> 2
